Commit message: Migrate from Polyhobbyist to RHR

File: test/testdata/basic_with_stl_mesh.urdf (robot description, URDF)
Before this commit: robot myfirst, 1 links, 0 joints
Links:
- link base_link: geometry visual mesh filename=https://raw.githubusercontent.com/Ranch-Hand-Robotics/babyl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

File: test/testdata/bb.urdf (robot description, URDF)
Before this commit: robot bb_head, 6 links, 5 joints
Links:
- link base_link: geometry visual mesh filename=https://raw.githubusercontent.com/Ranch-Hand-Robotics/bb_de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 scale=0.00001 0.00001 0.00001

File: test/testdata/mule.urdf (robot description, URDF)
Before this commit: robot mule, 7 links, 6 joints
Links:
- link left_front_wheel_link: geometry collision cylinder length=0.0889 radius=0.127; visual mesh filename=https://raw.githubusercontent.com/Ranch-Hand-Robotics/babyl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
- link left_mid_wheel_link: geometry collision cylinder length=0.0889 radius=0.127; visual mesh filename=https://raw.githubusercontent.com/Ranch-Hand-Robotics/babyl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
- link left_rear_wheel_link: geometry collision cylinder length=0.0889 radius=0.127; visual mesh filename=https://raw.githubusercontent.com/Ranch-Hand-Robotics/babyl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
- link right_front_wheel_link: geometry collision cylinder length=0.0889 radius=0.127; visual mesh filename=https://raw.githubusercontent.com/Ranch-Hand-Robotics/babyl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
- link right_mid_wheel_link: geometry collision cylinder length=0.0889 radius=0.127; visual mesh filename=https://raw.githubusercontent.com/Ranch-Hand-Robotics/babyl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
- link right_rear_wheel_link: geometry collision cylinder length=0.0889 radius=0.127; visual mesh filename=https://raw.githubusercontent.com/Ranch-Hand-Robotics/babyl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
