Commit message: Fix mule

File: test/testdata/mule.urdf (robot description, URDF)
Before this commit: robot mule, 7 links, 6 joints
Links:
- added link chassis_link; collision box size=0.508 0.7747 0.0762; visual box size=0.508 0.7747 0.0762
- link base_link: mass None -> 0.001; geometry 
Joints:
- added joint base_to_chassis: type fixed, parent base_link, child chassis_link, origin xyz=0 0 0.127 rpy=0 0 0
- joint left_front_wheel: parent base_link -> chassis_link
- joint left_mid_wheel: parent base_link -> chassis_link
- joint left_rear_wheel: parent base_link -> chassis_link
- joint right_front_wheel: parent base_link -> chassis_link
- joint right_mid_wheel: parent base_link -> chassis_link
- joint right_rear_wheel: parent base_link -> chassis_link

Commit message: Fix mule offset

File: test/testdata/mule.urdf (robot description, URDF)
Before this commit: robot mule, 8 links, 7 joints
Joints:
- joint base_to_chassis: origin xyz=0 0 0.127 rpy=0 0 0 -> xyz=0 0 0.527 rpy=0 0 0
